Commit message: small tweaks to paramsams

File: xarm_description/urdf/camera/realsense_d435i.urdf.xacro (robot description, xacro)
@@ -15,6 +15,11 @@
         origin_rpy="0 0 0" />
     </link>
+    <link name="${prefix}camera_link"></link>
+    <joint name="${prefix}camera_link_joint" type="fixed">
+      <parent link="${prefix}link_eef" />
+      <child link="${prefix}camera_link" />
+      <origin xyz="0.06746 -0.0175 0.0237" rpy="${M_PI} ${-M_PI/2} 0" />
+    </joint>
     <xacro:if value="${add_d435i_links}">
-      <link name="${prefix}camera_link"></link>
       <link name="${prefix}camera_depth_frame"></link>
       <link name="${prefix}camera_depth_optical_frame"></link>
@@ -25,9 +30,4 @@
       <link name="${prefix}camera_right_ir_frame"></link>
       <link name="${prefix}camera_right_ir_optical_frame"></link>
-      <joint name="${prefix}camera_link_joint" type="fixed">
-        <parent link="${prefix}link_eef" />
-        <child link="${prefix}camera_link" />
-        <origin xyz="0.06746 -0.0175 0.0237" rpy="${M_PI} ${-M_PI/2} 0" />
-      </joint>
       <joint name="${prefix}camera_depth_joint" type="fixed">
         <parent link="${prefix}camera_link" />

Commit message: updating camera mount thickness

File: xarm_description/urdf/camera/realsense_d435i.urdf.xacro (robot description, xacro)
@@ -15,6 +15,11 @@
         origin_rpy="0 0 0" />
     </link>
+    <link name="${prefix}camera_link"></link>
+    <joint name="${prefix}camera_link_joint" type="fixed">
+      <parent link="${prefix}link_eef" />
+      <child link="${prefix}camera_link" />
+      <origin xyz="0.06746 -0.0175 0.0337" rpy="${M_PI} ${-M_PI/2} 0" />
+    </joint>
     <xacro:if value="${add_d435i_links}">
-      <link name="${prefix}camera_link"></link>
       <link name="${prefix}camera_depth_frame"></link>
       <link name="${prefix}camera_depth_optical_frame"></link>

Commit message: updating camera mount thickness

File: xarm_description/urdf/camera/realsense_d435i.urdf.xacro (robot description, xacro)
@@ -19,5 +19,5 @@
       <parent link="${prefix}link_eef" />
       <child link="${prefix}camera_link" />
-      <origin xyz="0.06746 -0.0175 0.0237" rpy="${M_PI} ${-M_PI/2} 0" />
+      <origin xyz="0.06746 -0.0175 0.0337" rpy="${M_PI} ${-M_PI/2} 0" />
     </joint>
     <xacro:if value="${add_d435i_links}">

File: xarm_description/urdf/xarm_device_macro.xacro (robot description, xacro)
@@ -50,4 +50,5 @@
     <xacro:include filename="$(find xarm_description)/urdf/common/common.material.xacro" />
     <xacro:common_material prefix="${prefix}"/>
+    <xacro:property name="M_PI" value="3.1415926535897931" />
     <!-- Specify Mesh file path -->
     <xacro:property name="mesh_suffix" value="${mesh_suffix}" scope="parent"/>
@@ -227,6 +228,10 @@
         <!-- Load XArm Gripper Model URDF -->
         <xacro:include filename="$(find xarm_description)/urdf/gripper/xarm_gripper_macro.xacro" />
-        <xacro:xarm_gripper_macro prefix="${prefix}" attach_to="${prefix}link_eef"
-          ros2_control_plugin="${ros2_control_plugin}" dof="${dof}" hard_interface="${hard_interface}" />
+        <xacro:if value="${add_realsense_d435i}">
+          <xacro:xarm_gripper_macro prefix="${prefix}" attach_to="${prefix}camera_link" attach_xyz="-0.0287 -0.0175 -0.06746" attach_rpy="0 ${M_PI/2} 0" ros2_control_plugin="${ros2_control_plugin}" dof="${dof}" hard_interface="${hard_interface}" />
+        </xacro:if>
+        <xacro:unless value="${add_realsense_d435i}">
+          <xacro:xarm_gripper_macro prefix="${prefix}" attach_to="${prefix}link_eef" ros2_control_plugin="${ros2_control_plugin}" dof="${dof}" hard_interface="${hard_interface}" />
+        </xacro:unless>
       </xacro:unless>
     </xacro:if>
